Commit message: clean up

File: sysid/assets/leap_hand/urdf/leap_hand_right.urdf (robot description, URDF)
Before this commit: robot leap_right, 22 links, 21 joints
Links:
- removed link dip
- removed link dip_2
- removed link dip_3
- removed link fingertip
- removed link fingertip_2
- removed link fingertip_3
- removed link index_tip_head
- removed link mcp_joint
- removed link mcp_joint_2
- removed link mcp_joint_3
- removed link middle_tip_head
- removed link palm_lower
- removed link pip
- removed link pip_2
- removed link pip_3
- removed link ring_tip_head
- removed link thumb_dip
- removed link thumb_fingertip
- removed link thumb_pip
- removed link thumb_temp_base
- removed link thumb_tip_head
- added link if_bs, mass 0.044000; collision box size=0.014000 0.020000 0.004000; collision box size=0.014000 0.020000 0.004000
- added link if_ds, mass 0.016000; collision box size=0.014000 0.022000 0.004000; collision box size=0.014000 0.022000 0.004000
- added link if_md, mass 0.037000; collision box size=0.014000 0.020000 0.004000; collision box size=0.014000 0.020000 0.004000
- added link if_px, mass 0.032000; collision box size=0.034000 0.026000 0.022000; visual mesh filename=../mjcf/assets/proximal.obj
- added link mf_bs, mass 0.044000; collision box size=0.014000 0.020000 0.004000; collision box size=0.014000 0.020000 0.004000
- added link mf_ds, mass 0.016000; collision box size=0.014000 0.022000 0.004000; collision box size=0.014000 0.022000 0.004000
- added link mf_md, mass 0.037000; collision box size=0.014000 0.020000 0.004000; collision box size=0.014000 0.020000 0.004000
- added link mf_px, mass 0.032000; collision box size=0.034000 0.026000 0.022000; visual mesh filename=../mjcf/assets/proximal.obj
- added link palm, mass 0.237000; collision box size=0.004000 0.036000 0.034000; collision box size=0.010000 0.120000 0.020000
- added link rf_bs, mass 0.044000; collision box size=0.014000 0.020000 0.004000; collision box size=0.014000 0.020000 0.004000
- added link rf_ds, mass 0.016000; collision box size=0.014000 0.022000 0.004000; collision box size=0.014000 0.022000 0.004000
- added link rf_md, mass 0.037000; collision box size=0.014000 0.020000 0.004000; collision box size=0.014000 0.020000 0.004000
- added link rf_px, mass 0.032000; collision box size=0.034000 0.026000 0.022000; visual mesh filename=../mjcf/assets/proximal.obj
- added link th_bs, mass 0.003000; collision box size=0.014000 0.004000 0.020000; collision box size=0.014000 0.004000 0.020000
- added link th_ds, mass 0.049000; collision box size=0.008000 0.024000 0.018000; collision box size=0.020000 0.004000 0.030000
- added link th_mp, mass 0.032000; collision box size=0.034000 0.026000 0.022000; visual mesh filename=../mjcf/assets/proximal.obj
- added link th_px, mass 0.038000; collision box size=0.010000 0.024000 0.018000; collision box size=0.014000 0.020000 0.004000
Joints:
- removed joint base_joint
- removed joint index_tip
- removed joint joint_0
- removed joint joint_1
- removed joint joint_10
- removed joint joint_11
- removed joint joint_12
- removed joint joint_13
- removed joint joint_14
- removed joint joint_15
- removed joint joint_2
- removed joint joint_3
- removed joint joint_4
- removed joint joint_5
- removed joint joint_6
- removed joint joint_7
- removed joint joint_8
- removed joint joint_9
- removed joint middle_tip
- removed joint ring_tip
- removed joint thumb_tip
- added joint base_palm_fixed: type fixed, parent base, child palm, origin xyz=0.057595 -0.033342 0.011278 rpy=3.141593 0.000000 0.000000
- added joint if_dip: type revolute, parent if_md, child if_ds, origin xyz=0.000000 -0.036100 0.000200 rpy=0.000000 0.000000 0.000000, axis 0.000000 0.000000 -1.000000, limit lower=-0.366000 upper=2.042000 effort=0.5 velocity=8
- added joint if_mcp: type revolute, parent palm, child if_bs, origin xyz=-0.007000 0.023000 -0.018700 rpy=1.570796 1.570796 0.000003, axis 0.000000 0.000000 -1.000000, limit lower=-0.314000 upper=2.230000 effort=0.5 velocity=8
- added joint if_pip: type revolute, parent if_px, child if_md, origin xyz=0.015000 0.014300 -0.013000 rpy=1.570796 -1.570796 -0.000003, axis 0.000000 0.000000 -1.000000, limit lower=-0.506000 upper=1.885000 effort=0.5 velocity=8
- added joint if_rot: type revolute, parent if_bs, child if_px, origin xyz=-0.012200 0.038100 0.014500 rpy=-1.570790 0.000000 1.570790, axis 0.000000 0.000000 -1.000000, limit lower=-1.047000 upper=1.047000 effort=0.5 velocity=8
- added joint mf_dip: type revolute, parent mf_md, child mf_ds, origin xyz=0.000000 -0.036100 0.000200 rpy=0.000000 0.000000 0.000000, axis 0.000000 0.000000 -1.000000, limit lower=-0.366000 upper=2.042000 effort=0.5 velocity=8
- added joint mf_mcp: type revolute, parent palm, child mf_bs, origin xyz=-0.007100 -0.022400 -0.018700 rpy=1.570796 1.570796 0.000003, axis 0.000000 0.000000 -1.000000, limit lower=-0.314000 upper=2.230000 effort=0.5 velocity=8
- added joint mf_pip: type revolute, parent mf_px, child mf_md, origin xyz=0.015000 0.014300 -0.013000 rpy=1.570796 -1.570796 -0.000003, axis 0.000000 0.000000 -1.000000, limit lower=-0.506000 upper=1.885000 effort=0.5 velocity=8
- added joint mf_rot: type revolute, parent mf_bs, child mf_px, origin xyz=-0.012200 0.038100 0.014500 rpy=-1.570790 0.000000 1.570790, axis 0.000000 0.000000 -1.000000, limit lower=-1.047000 upper=1.047000 effort=0.5 velocity=8
- added joint rf_dip: type revolute, parent rf_md, child rf_ds, origin xyz=0.000000 -0.036090 0.000200 rpy=0.000000 0.000000 0.000000, axis 0.000000 0.000000 -1.000000, limit lower=-0.366000 upper=2.042000 effort=0.5 velocity=8
- added joint rf_mcp: type revolute, parent palm, child rf_bs, origin xyz=-0.007090 -0.067800 -0.018700 rpy=1.570796 1.570796 0.000003, axis 0.000000 0.000000 -1.000000, limit lower=-0.314000 upper=2.230000 effort=0.5 velocity=8
- added joint rf_pip: type revolute, parent rf_px, child rf_md, origin xyz=0.015000 0.014300 -0.013000 rpy=1.570796 -1.570796 -0.000003, axis 0.000000 0.000000 -1.000000, limit lower=-0.506000 upper=1.885000 effort=0.5 velocity=8
- added joint rf_rot: type revolute, parent rf_bs, child rf_px, origin xyz=-0.012200 0.038100 0.014500 rpy=-1.570790 0.000000 1.570790, axis 0.000000 0.000000 -1.000000, limit lower=-1.047000 upper=1.047000 effort=0.5 velocity=8
- added joint th_axl: type revolute, parent th_mp, child th_bs, origin xyz=0.000000 0.014300 -0.013000 rpy=1.570796 -1.570796 -0.000003, axis 0.000000 0.000000 -1.000000, limit lower=-0.349000 upper=2.094000 effort=0.5 velocity=8
- added joint th_cmc: type revolute, parent palm, child th_mp, origin xyz=-0.069300 -0.001200 -0.021600 rpy=0.000000 1.570796 0.000000, axis 0.000000 0.000000 -1.000000, limit lower=-0.349000 upper=2.094000 effort=0.5 velocity=8
- added joint th_ipl: type revolute, parent th_px, child th_ds, origin xyz=0.000000 0.046600 0.000200 rpy=0.000000 0.000000 3.141590, axis 0.000000 0.000000 -1.000000, limit lower=-1.340000 upper=1.880000 effort=0.5 velocity=8
- added joint th_mcp: type revolute, parent th_bs, child th_px, origin xyz=0.000000 0.014500 -0.017000 rpy=-1.570791 0.000000 0.000000, axis 0.000000 0.000000 -1.000000, limit lower=-0.470000 upper=2.443000 effort=0.5 velocity=8
